Commit message: Update camera.xacro

File: description/camera.xacro (robot description, xacro)
@@ -4,5 +4,5 @@
         <parent link="chassis"/>
         <child link="camera_link"/>
-        <origin xyz="0.276 0 0.181" rpy="0 0.18 0"/>
+        <origin xyz="0.70 0.35 0.181" rpy="0 0 0"/>
     </joint>
     <link name="camera_link">

Commit message: Update camera.xacro

File: description/camera.xacro (robot description, xacro)
@@ -4,5 +4,5 @@
         <parent link="chassis"/>
         <child link="camera_link"/>
-        <origin xyz="0.70 0.35 0.181" rpy="0 0 0"/>
+        <origin xyz="0.31 0.035 0.05" rpy="0 0 0"/>
     </joint>
     <link name="camera_link">

Commit message: Update camera.xacro

File: description/camera.xacro (robot description, xacro)
@@ -4,5 +4,5 @@
         <parent link="chassis"/>
         <child link="camera_link"/>
-        <origin xyz="0.31 0.035 0.05" rpy="0 0 0"/>
+        <origin xyz="0.31 -0.035 0.05" rpy="0 0 0"/>
     </joint>
     <link name="camera_link">
@@ -14,7 +14,7 @@
         </visual>
         <visual>
-            <origin xyz="0 0 -0.05"/>
+            <origin xyz="0 0 0"/>
             <geometry>
-                <cylinder radius="0.002" length="0.1"/>
+                <cylinder radius="0.002" length="0.01"/>
             </geometry>
             <material name="black"/>
